Commit message: added new accessories

File: husky_custom_description/urdf/husky_custom_description.urdf.xacro (robot description, xacro)
@@ -1,4 +1,23 @@
 <?xml version="1.0"?>
 <robot xmlns:xacro="http://ros.org/wiki/xacro" name="camera_mount">
+<xacro:arg name="arm" default="gen3" />
+<xacro:arg name="dof" default="7" />
+<xacro:arg name="vision" default="true" />
+<xacro:arg name="gripper" default="robotiq_2f_85" />
+<xacro:arg name="sim" default="false" />
+<xacro:arg name="prefix" default="kinova_arm_" />
+<xacro:include filename="$(find kortex_description)/robots/kortex_robot.xacro" />
+<xacro:if value="$(optenv HUSKY_KINOVA 0)">
+    <xacro:load_robot arm="$(arg arm)" gripper="$(arg gripper)" dof="$(arg dof)" vision="$(arg vision)" sim="$(arg sim)" prefix="$(arg prefix)" />
+    <joint name="arm_mount_joint" type="fixed">
+        <origin xyz="$(optenv HUSKY_KINOVA_XYZ -0.105 0.0 0.0)" rpy="$(optenv HUSKY_KINOVA_RPY 0 0 0)" />
+        <parent link="top_plate_front_link" />
+        <child link="kinova_arm_base_link" />
+    </joint>
+</xacro:if>
+<xacro:if value="$(optenv RPLIDAR 0)">
+    <xacro:include filename="$(find husky_description)/urdf/accessories/rplidar.urdf.xacro" />
+    <xacro:rplidar parent_link="top_plate_front_link" xyz="$(optenv RPLIDAR_LASER_XYZ 0 0 0)" rpy="$(optenv RPLIDAR_LASER_RPY 0 0 0)"/>
+</xacro:if>
 <xacro:property name="camera_mount_height" value="0.12" />
 <xacro:property name="camera_mount_spacing" value="0.12" />

Commit message: added collision for sensor arch and camera

File: husky_custom_description/urdf/husky_custom_description.urdf.xacro (robot description, xacro)
@@ -7,4 +7,19 @@
 <xacro:arg name="sim" default="false" />
 <xacro:arg name="prefix" default="kinova_arm_" />
+<xacro:if value="$(optenv HUSKY_SENSOR_ARCH 0)">
+    <link name="sensor_arch_collision_link">
+        <collision>
+            <geometry>
+                <box size="0.15 0.55 0.8"/>
+            </geometry>
+            <origin xyz="0 0 0.4" rpy="0 0 0"/>
+        </collision>
+    </link>
+    <joint name="sensor_arch_collision_joint" type="fixed">
+        <origin xyz="0 0 0" rpy="0 0 0" />
+        <parent link="sensor_arch_base_link" />
+        <child link="sensor_arch_collision_link" />
+    </joint>
+</xacro:if>
 <xacro:include filename="$(find kortex_description)/robots/kortex_robot.xacro" />
 <xacro:if value="$(optenv HUSKY_KINOVA 0)">
